File: Homekey.kicad_sch (KiCad schematic)
At the start: 0 parts

Commit message: Added Revs + PDF
Other:
- title: (none) -> Homekey PCB ESP32C3
Changed lines of the file:
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@@
 	(generator_version "8.0")
 	(paper "A4")
+	(title_block
+		(title "Homekey PCB ESP32C3")
+		(date "2024-07-03")
+		(rev "Rev A")
+	)
 	(sheet
 		(at 100.33 31.75)
