File: NFC.kicad_sch (KiCad schematic)
At the start: 36 parts, among them J1 Hirose, U2 PN5321A3HN_C1xx, Y1 27.12MHz

Commit message: Added Revs + PDF
Other:
- title: (none) -> Homekey PCB ESP32C3
Changed lines of the file:
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@@
 	(generator_version "8.0")
 	(paper "A4")
+	(title_block
+		(title "Homekey PCB ESP32C3")
+		(date "2024-07-03")
+		(rev "Rev A")
+	)
 	(junction
 		(at 219.71 106.68)

Commit message: Start of layout
Parts:
- C1, C14, C15, C16, C17, C20, C21, C23, C4: footprint RevK:C_0603 -> Capacitor_SMD_AKL:C_0603_1608Metric; symbol Device:C -> PCM_Capacitor_US_AKL:C_0603
- C18, C19, C5, C7, C8, C9: footprint Capacitor_SMD:C_0603_1608Metric -> Capacitor_SMD_AKL:C_0603_1608Metric; symbol Device:C -> PCM_Capacitor_US_AKL:C_0603
- C22: footprint RevK:C_0603 -> Capacitor_SMD:C_0603_1608Metric
- JP1, JP2: footprint (none) -> Jumper:SolderJumper-3_P2.0mm_Open_TrianglePad1.0x1.5mm
- L1, L2: footprint RevK:L_1206_1008 -> Inductor_SMD:L_0805_2012Metric
- R1, R2, R3, R4, R5: footprint RevK:R_0603 -> Resistor_SMD_AKL:R_0603_1608Metric; symbol Device:R -> PCM_Resistor_AKL:R_0603
- TP1: footprint RevK:PN532-RF-Test -> TestPoint:TestPoint_2Pads_Pitch2.54mm_Drill0.8mm
- Y1: footprint RevK:Crystal-3.2x2.5 -> Crystal:Crystal_SMD_3225-4Pin_3.2x2.5mm
Connections:
- net NFC_TX2: now reaches L1.2, TP1.2
- net NFC_TX2: now also U2.6 (TX2); no longer U2.4 (TX1)
- net NFC_TX1: now reaches L2.1, TP1.1
- net NFC_TX1: now also U2.4 (TX1); no longer U2.6 (TX2)
- net NFC_RX1: now reaches C16.2, C18.2, C20.1, L1.1
- net NFC_RX1: now also R3.2
- net at C17.2, C19.1, C21.1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: no longer R3.2
Other:
- moved on the sheet: C16, C17, C18, C19, C20, C21, C22, C23, J1, L1, L2, R4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

Commit message: Finished rev A PCB V 0.1
Parts:
- removed TP1: TestPoint_2Pole, TestPoint:TestPoint_2Pads_Pitch2.54mm_Drill0.8mm, symbol Connector:TestPoint_2Pole
- renumbered JP1 to SEL0, JP2 to SEL1
Changed lines of the file:
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@@
 	)
 	(junction
-		(at 210.82 121.92)
-		(diameter 0)
-		(color 0 0 0 0)
-	)
-	(junction
 		(at 82.55 138.43)
 		(diameter 0)
@@
 	)
 	(junction
-		(at 210.82 142.24)
-		(diameter 0)
-		(color 0 0 0 0)
-	)
-	(junction
 		(at 139.7 36.83)
 		(diameter 0)
@@
 	(wire
 		(pts
-			(xy 210.82 142.24) (xy 209.55 142.24)
-		)
-		(stroke
-			(width 0)
-			(type default)
-		)
-	)
-	(wire
-		(pts
 			(xy 240.03 142.24) (xy 234.95 142.24)
 		)
@@
 	(wire
 		(pts
-			(xy 217.17 121.92) (xy 210.82 121.92)
+			(xy 209.55 121.92) (xy 217.17 121.92)
 		)
 		(stroke
@@
 	(wire
 		(pts
-			(xy 210.82 127) (xy 210.82 121.92)
-		)
-		(stroke
-			(width 0)
-			(type default)
-		)
-	)
-	(wire
-		(pts
 			(xy 189.23 53.34) (xy 190.5 53.34)
 		)
@@
 	(wire
 		(pts
-			(xy 217.17 142.24) (xy 210.82 142.24)
+			(xy 209.55 142.24) (xy 217.17 142.24)
 		)
 		(stroke
@@
 	(wire
 		(pts
-			(xy 210.82 142.24) (xy 210.82 137.16)
-		)
-		(stroke
-			(width 0)
-			(type default)
-		)
-	)
-	(wire
-		(pts
 			(xy 106.68 133.35) (xy 106.68 130.81)
 		)
@@
 	(wire
 		(pts
-			(xy 210.82 121.92) (xy 209.55 121.92)
-		)
-		(stroke
-			(width 0)
-			(type default)
-		)
-	)
-	(wire
-		(pts
 			(xy 134.62 151.13) (xy 134.62 153.67)
 		)
@@
 		(dnp no)
 		(fields_autoplaced yes)
-		(property "Reference" "JP2"
+		(property "Reference" "SEL1"
 			(at 184.15 46.99 0)
 			(effects
@@
 			(project "Homekey"
 				(path "/8ef12b84-4556-413e-8e5a-ce52402aeac0/18dde409-6af5-4dc2-8e7a-03cef80bd424"
-					(reference "JP2")
+					(reference "SEL1")
 					(unit 1)
 				)
@@
 		(dnp no)
 		(fields_autoplaced yes)
-		(property "Reference" "JP1"
+		(property "Reference" "SEL0"
 			(at 184.15 35.56 0)
 			(effects
@@
 			(project "Homekey"
 				(path "/8ef12b84-4556-413e-8e5a-ce52402aeac0/18dde409-6af5-4dc2-8e7a-03cef80bd424"
-					(reference "JP1")
+					(reference "SEL0")
 					(unit 1)
 				)
@@
 					(unit 1)
 				)
-			)
-		)
-	)
-	(symbol
-		(lib_id "Connector:TestPoint_2Pole")
-		(at 210.82 132.08 90)
-		(unit 1)
-		(exclude_from_sim no)
-		(in_bom no)
-		(on_board yes)
-		(dnp no)
-		(property "Reference" "TP1"
-			(at 215.138 132.334 90)
-			(effects
-				(font
-					(size 1.27 1.27)
-				)
-				(justify left)
-			)
-		)
-		(property "Value" "TestPoint_2Pole"
-			(at 209.3468 130.937 90)
-			(effects
-				(font
-					(size 1.27 1.27)
-				)
-				(justify left)
-				(hide yes)
-			)
-		)
-		(property "Footprint" "TestPoint:TestPoint_2Pads_Pitch2.54mm_Drill0.8mm"
-			(at 210.82 132.08 0)
-			(effects
-				(font
-					(size 1.27 1.27)
-				)
-				(hide yes)
-			)
-		)
-		(property "Datasheet" "~"
-			(at 210.82 132.08 0)
-			(effects
-				(font
-					(size 1.27 1.27)
-				)
-				(hide yes)
-			)
-		)
-		(property "Description" ""
-			(at 210.82 132.08 0)
-			(effects
-				(font
-					(size 1.27 1.27)
-				)
-				(hide yes)
-			)
-		)
-		(property "Note" "No part, PCB printed"
-			(at 210.82 132.08 90)
-			(effects
-				(font
-					(size 1.27 1.27)
-				)
-				(hide yes)
-			)
-		)
-		(pin "1"
-		)
-		(pin "2"
-		)
-		(instances
-			(project "Homekey"
-				(path "/8ef12b84-4556-413e-8e5a-ce52402aeac0/18dde409-6af5-4dc2-8e7a-03cef80bd424"
-					(reference "TP1")
-					(unit 1)
-				)
