File: Homekey.kicad_pcb (KiCad board)
At the start: 2 copper layers, 75 x 40 mm, 71 parts, among them J1 Hirose, J2 Screw_Terminal_01x02, J3 USB_C_Receptacle_USB2.0_16P, U1 ESP32-C3-WROOM-02, U2 PN5321A3HN_C1xx, U3 MAX17501AxTB, U4 TLV75533PDRV, Y1 27.12MHz

Commit message: Finished rev A PCB V 0.1
Parts:
- removed C29: 10uF, Capacitor_SMD:C_0805_2012Metric
- added GND1: TestPoint, TestPoint:TestPoint_THTPad_1.5x1.5mm_Drill0.7mm, F.Cu at (156.1, 85.7)
- moved C26 206.3 mm to (182.0, 77.8)
- moved C2 204.3 mm to (183.2, 81.3), turned to 90 degrees
- moved D1 203.5 mm to (191.0, 77.0)
- moved C28 202.9 mm to (180.3, 85.1), turned to 180 degrees
- moved C24 202.6 mm to (179.0, 77.8), turned to 180 degrees
- moved C3 201.9 mm to (187.0, 82.3), turned to -90 degrees
- moved J2 200.8 mm to (191.8, 84.6), turned to 90 degrees
- moved C25 200.8 mm to (185.0, 82.3), turned to -90 degrees
- moved C27 197.1 mm to (180.5, 83.1)
- moved U3 196.3 mm to (180.5, 80.3), turned to 180 degrees
- moved C30 183.3 mm to (165.0, 86.3), turned to 180 degrees
- moved C31 182.5 mm to (162.2, 84.1), turned to -90 degrees
- moved L3 181.7 mm to (175.5, 82.1), turned to -90 degrees
- moved R6 177.9 mm to (163.5, 92.1)
- moved R7 177.7 mm to (163.5, 95.3)
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- renumbered JP1 to SEL0, JP2 to SEL1
Routing:
- net +3.3V: track 4.47 -> 135.9 mm, vias 0 -> 15
- net SCL: track 0.00 -> 68.8 mm, vias 0 -> 7
- net SCK_NFC: track 0.00 -> 62.3 mm, vias 0 -> 4
- net MISO_NFC: track 0.00 -> 57.3 mm, vias 0 -> 6
- net RST_NFC: track 0.00 -> 51.8 mm, vias 0 -> 4
- net GND: track 21.7 -> 72.1 mm, vias 0 -> 76
- net LED_G: track 0.00 -> 47.2 mm, vias 0 -> 2
- net IRQ_NFC: track 0.00 -> 45.7 mm, vias 0 -> 4
- net SDA: track 0.00 -> 43.1 mm, vias 0 -> 5
- net LED_R: track 0.00 -> 37.5 mm
- net Net-(D1-A): track 0.00 -> 34.2 mm
- net Net-(U1-IO21/TXD): track 0.00 -> 27.7 mm, vias 0 -> 2
- net Net-(U2-AVDD): track 0.00 -> 22.8 mm, vias 0 -> 4
- net Net-(U1-IO20/RXD): track 0.00 -> 21.2 mm, vias 0 -> 2
- net LED_B: track 0.00 -> 20.9 mm, vias 0 -> 2
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- added copper zone on F.Cu, net +3.3V
- added copper zone on B.Cu, net GND
- added copper zone on F.Cu, net GND
- added copper zone on F.Cu, net Net-(U3-LX)
- added copper zone on F.Cu, net VIN
Other:
- board size 75 x 40 mm -> 41.6 x 47.3 mm
- board text added: "ESP HomeKey Ver 0.1A"
- board text added: "Generator"
- board text added: "Made to Impress Build to Excel"
- board text added: "Nightmare"

Commit message: Adding gerbers + BOM
Parts:
- D1: footprint Fuse:Fuseholder_Littelfuse_Nano2_157x -> Diode_SMD:D_SOD-123
Routing:
- net Net-(D1-A): track 34.2 -> 33.4 mm
